File: profane_geometry/geo_core.sch (KiCad schematic (older format))
At the start: 54 parts, among them Q1 MMBF4416A, U2 TL074, U3 TL074, U4 TL074

Commit message: update .gitignore, current kicad project
Parts:
- C10: renamed from C7; footprint Capacitor_SMD:C_0805_2012Metric_Pad1.18x1.45mm_HandSolder -> Capacitor_SMD:C_0805_2012Metric; MFG Part No. (none) -> 08055A220KAT4A
- C11: renamed from C8; value 10uF -> 4.7uF; footprint Capacitor_SMD:C_0805_2012Metric_Pad1.18x1.45mm_HandSolder -> Capacitor_SMD:C_0805_2012Metric; MFG Part No. (none) -> 08053C475KAT2A
- C12: renamed from C9; footprint Capacitor_SMD:C_1206_3216Metric_Pad1.33x1.80mm_HandSolder -> Capacitor_SMD:C_0805_2012Metric; MFG Part No. (none) -> 08055C104KAT4A
- C13: renamed from C10; footprint Capacitor_SMD:C_1206_3216Metric_Pad1.33x1.80mm_HandSolder -> Capacitor_SMD:C_0805_2012Metric; MFG Part No. (none) -> 08055C104KAT4A
- C14: renamed from C11; footprint Capacitor_SMD:C_1206_3216Metric_Pad1.33x1.80mm_HandSolder -> Capacitor_SMD:C_0805_2012Metric; MFG Part No. (none) -> 08055C104KAT4A
- C15: renamed from C12; footprint Capacitor_SMD:C_1206_3216Metric_Pad1.33x1.80mm_HandSolder -> Capacitor_SMD:C_0805_2012Metric; MFG Part No. (none) -> 08055C104KAT4A
- C16: renamed from C13; footprint Capacitor_SMD:C_1206_3216Metric_Pad1.33x1.80mm_HandSolder -> Capacitor_SMD:C_0805_2012Metric; MFG Part No. (none) -> 08055C104KAT4A
- C17: renamed from C14; footprint Capacitor_SMD:C_1206_3216Metric_Pad1.33x1.80mm_HandSolder -> Capacitor_SMD:C_0805_2012Metric; MFG Part No. (none) -> 08055C104KAT4A
- C7: renamed from C4; footprint Capacitor_SMD:C_0805_2012Metric_Pad1.18x1.45mm_HandSolder -> Capacitor_SMD:C_0805_2012Metric; MFG Part No. (none) -> 08055C473KAT2A
- C8: renamed from C5; footprint Capacitor_SMD:C_0805_2012Metric_Pad1.18x1.45mm_HandSolder -> Capacitor_SMD:C_0805_2012Metric; MFG Part No. (none) -> 08055C222KAT2A
- C9: renamed from C6; value 10uF -> 1uF; footprint Capacitor_SMD:C_0805_2012Metric_Pad1.18x1.45mm_HandSolder -> Capacitor_SMD:C_0805_2012Metric; MFG Part No. (none) -> 0805DC105KAT2A
- D4: renamed from D3; MFG Part No. (none) -> 1N5819HWQ-7-F
- D5: renamed from D4; MFG Part No. (none) -> 1N5819HWQ-7-F
- Q1: MFG Part No. (none) -> MMBF4416A
- R10: renamed from R9; footprint Resistor_SMD:R_1206_3216Metric_Pad1.30x1.75mm_HandSolder -> Resistor_SMD:R_0805_2012Metric; MFG Part No. (none) -> RMCF0805FT1M00
- R11: renamed from R10; footprint Resistor_SMD:R_1206_3216Metric_Pad1.30x1.75mm_HandSolder -> Resistor_SMD:R_0805_2012Metric; MFG Part No. (none) -> RMCF0805FT10K0
- R12: renamed from R11; footprint Resistor_SMD:R_0805_2012Metric_Pad1.20x1.40mm_HandSolder -> Resistor_SMD:R_0805_2012Metric; MFG Part No. (none) -> RMCF0805FT1K00
- R13: renamed from R12; footprint Resistor_SMD:R_0805_2012Metric_Pad1.20x1.40mm_HandSolder -> Resistor_SMD:R_0805_2012Metric; MFG Part No. (none) -> RMCF0805FT7K15
- R14: renamed from R13; footprint Resistor_SMD:R_0805_2012Metric_Pad1.20x1.40mm_HandSolder -> Resistor_SMD:R_0805_2012Metric; MFG Part No. (none) -> RMCF0805FT2K87
- R15: renamed from R14; footprint Resistor_SMD:R_1206_3216Metric_Pad1.30x1.75mm_HandSolder -> Resistor_SMD:R_0805_2012Metric; MFG Part No. (none) -> RMCF0805FT4K12
- R16: renamed from R15; footprint Resistor_SMD:R_1206_3216Metric_Pad1.30x1.75mm_HandSolder -> Resistor_SMD:R_0805_2012Metric; MFG Part No. (none) -> RMCF0805FT10K0
- R17: renamed from R16; footprint Resistor_SMD:R_1206_3216Metric_Pad1.30x1.75mm_HandSolder -> Resistor_SMD:R_0805_2012Metric; MFG Part No. (none) -> RMCF0805FT10K0
- R18: renamed from R17; footprint Resistor_SMD:R_0805_2012Metric_Pad1.20x1.40mm_HandSolder -> Resistor_SMD:R_0805_2012Metric; MFG Part No. (none) -> RMCF0805FT1K00
- R19: renamed from R18; footprint Resistor_SMD:R_1206_3216Metric_Pad1.30x1.75mm_HandSolder -> Resistor_SMD:R_0805_2012Metric; MFG Part No. (none) -> RMCF0805FT3K57
- R2: renamed from R1; footprint Resistor_SMD:R_1206_3216Metric_Pad1.30x1.75mm_HandSolder -> Resistor_SMD:R_0805_2012Metric; MFG Part No. (none) -> RMCF0805FT10K0
- R20: renamed from R19; footprint Resistor_SMD:R_1206_3216Metric_Pad1.30x1.75mm_HandSolder -> Resistor_SMD:R_0805_2012Metric; MFG Part No. (none) -> RMCF0805FT10K0
- R21: renamed from R20; footprint Resistor_SMD:R_0805_2012Metric_Pad1.20x1.40mm_HandSolder -> Resistor_SMD:R_0805_2012Metric; MFG Part No. (none) -> RMCF0805FT169K
- R22: renamed from R21; footprint Resistor_SMD:R_1206_3216Metric_Pad1.30x1.75mm_HandSolder -> Resistor_SMD:R_0805_2012Metric; MFG Part No. (none) -> RMCF0805FT47K0
- R23: renamed from R22; value 33k -> 49.9k; footprint Resistor_SMD:R_1206_3216Metric_Pad1.30x1.75mm_HandSolder -> Resistor_SMD:R_0805_2012Metric; MFG Part No. (none) -> RMCF0805FT49K9
- R24: renamed from R23; footprint Resistor_SMD:R_1206_3216Metric_Pad1.30x1.75mm_HandSolder -> Resistor_SMD:R_0805_2012Metric; MFG Part No. (none) -> RMCF0805FT240K
- R25: renamed from R24; footprint Resistor_SMD:R_1206_3216Metric_Pad1.30x1.75mm_HandSolder -> Resistor_SMD:R_0805_2012Metric; MFG Part No. (none) -> RMCF0805FT10K0
- R26: renamed from R25; footprint Resistor_SMD:R_1206_3216Metric_Pad1.30x1.75mm_HandSolder -> Resistor_SMD:R_0805_2012Metric; MFG Part No. (none) -> RMCF0805FT47K0
- R27: renamed from R26; footprint Resistor_SMD:R_1206_3216Metric_Pad1.30x1.75mm_HandSolder -> Resistor_SMD:R_0805_2012Metric; MFG Part No. (none) -> RMCF0805FT22K0
- R28: renamed from R27; footprint Resistor_SMD:R_0805_2012Metric_Pad1.20x1.40mm_HandSolder -> Resistor_SMD:R_0805_2012Metric; MFG Part No. (none) -> RMCF0805FT8K25
- R29: renamed from R28; footprint Resistor_SMD:R_0805_2012Metric_Pad1.20x1.40mm_HandSolder -> Resistor_SMD:R_0805_2012Metric; MFG Part No. (none) -> RMCF0805FT1K00
- R3: renamed from R2; footprint Resistor_SMD:R_1206_3216Metric_Pad1.30x1.75mm_HandSolder -> Resistor_SMD:R_0805_2012Metric; MFG Part No. (none) -> RMCF0805FT10K0
- R30: renamed from R29; footprint Resistor_SMD:R_0805_2012Metric_Pad1.20x1.40mm_HandSolder -> Resistor_SMD:R_0805_2012Metric; MFG Part No. (none) -> RMCF0805FT30K1
- R31: renamed from R30; footprint Resistor_SMD:R_1206_3216Metric_Pad1.30x1.75mm_HandSolder -> Resistor_SMD:R_0805_2012Metric; MFG Part No. (none) -> RMCF0805FT10K0
- R32: renamed from R31; footprint Resistor_SMD:R_0805_2012Metric_Pad1.20x1.40mm_HandSolder -> Resistor_SMD:R_0805_2012Metric; MFG Part No. (none) -> RMCF0805FT1K00
- R33: renamed from R32; value 47k -> 100k; footprint Resistor_SMD:R_1206_3216Metric_Pad1.30x1.75mm_HandSolder -> Resistor_SMD:R_0805_2012Metric; MFG Part No. (none) -> RMCF0805FT100K
- R34: renamed from R33; footprint Resistor_SMD:R_1206_3216Metric_Pad1.30x1.75mm_HandSolder -> Resistor_SMD:R_0805_2012Metric; MFG Part No. (none) -> RMCF0805FT10K0
- R4: renamed from R3; footprint Resistor_SMD:R_1206_3216Metric_Pad1.30x1.75mm_HandSolder -> Resistor_SMD:R_0805_2012Metric; MFG Part No. (none) -> RMCF0805FT10K0
- R5: renamed from R4; footprint Resistor_SMD:R_1206_3216Metric_Pad1.30x1.75mm_HandSolder -> Resistor_SMD:R_0805_2012Metric; MFG Part No. (none) -> RMCF0805FT10K0
- R6: renamed from R5; value 5.9k -> 5.6k; footprint Resistor_SMD:R_0805_2012Metric_Pad1.20x1.40mm_HandSolder -> Resistor_SMD:R_0805_2012Metric; MFG Part No. (none) -> RMCF0805FT5K60
- R7: renamed from R6; footprint Resistor_SMD:R_1206_3216Metric_Pad1.30x1.75mm_HandSolder -> Resistor_SMD:R_0805_2012Metric; MFG Part No. (none) -> RMCF0805FT10K0
- R8: renamed from R7; footprint Resistor_SMD:R_0805_2012Metric_Pad1.20x1.40mm_HandSolder -> Resistor_SMD:R_0805_2012Metric; MFG Part No. (none) -> RMCF0805FT1K00
- R9: renamed from R8; footprint Resistor_SMD:R_1206_3216Metric_Pad1.30x1.75mm_HandSolder -> Resistor_SMD:R_0805_2012Metric; MFG Part No. (none) -> RMCF0805FT10K0
- TP1, TP2, TP3, TP4: footprint TestPoint:TestPoint_Pad_D2.0mm -> TestPoint:TestPoint_Pad_D1.0mm
- U3: renamed from U2; footprint Package_SO:SOIC-14_3.9x8.7mm_P1.27mm -> Package_SO:SSOP-14_5.3x6.2mm_P0.65mm; MFG Part No. (none) -> TL074CDBR
- U4: renamed from U3; footprint Package_SO:SOIC-14_3.9x8.7mm_P1.27mm -> Package_SO:SSOP-14_5.3x6.2mm_P0.65mm; MFG Part No. (none) -> TL074CDBR
- U5: renamed from U4; footprint Package_SO:SOIC-14_3.9x8.7mm_P1.27mm -> Package_SO:SSOP-14_5.3x6.2mm_P0.65mm; MFG Part No. (none) -> TL074CDBR
Other:
- note added: "0v -> 5v"
- note added: "Output here should be right around 17vpp. \nThe Tri-pre signal is an -9V -> +9V.\nThis circuit is a comparator that handles pwm, \nand a 1V separation between the two seems to give \na nice range from 2% @ 0V -> 98% @ 17V duty cycles."
- note removed: "0v -> 3.3v"
