File: profane_geometry/inputs.sch (KiCad schematic (older format))
At the start: 14 parts, among them U7 MCP6002-xSN, U8 MCP4728

Commit message: update .gitignore, current kicad project
Parts:
- C28: renamed from C18; footprint Capacitor_SMD:C_0805_2012Metric_Pad1.18x1.45mm_HandSolder -> Capacitor_SMD:C_0805_2012Metric; MFG Part No. (none) -> 08055C472KAT2A
- C29: renamed from C19; footprint Capacitor_SMD:C_0805_2012Metric_Pad1.18x1.45mm_HandSolder -> Capacitor_SMD:C_0805_2012Metric; MFG Part No. (none) -> 08055C222KAT2A
- C30: renamed from C20; footprint Capacitor_SMD:C_1206_3216Metric_Pad1.33x1.80mm_HandSolder -> Capacitor_SMD:C_0805_2012Metric; MFG Part No. (none) -> 08055C104KAT4A
- C31: renamed from C21; footprint Capacitor_SMD:C_1206_3216Metric_Pad1.33x1.80mm_HandSolder -> Capacitor_SMD:C_0805_2012Metric; MFG Part No. (none) -> 08055C104KAT4A
- R62: renamed from R50; footprint Resistor_SMD:R_0805_2012Metric_Pad1.20x1.40mm_HandSolder -> Resistor_SMD:R_0805_2012Metric; MFG Part No. (none) -> RMCF0805FT100K
- R63: renamed from R51; footprint Resistor_SMD:R_1206_3216Metric_Pad1.30x1.75mm_HandSolder -> Resistor_SMD:R_0805_2012Metric; MFG Part No. (none) -> RMCF0805FT240K
- R64: renamed from R52; footprint Resistor_SMD:R_0805_2012Metric_Pad1.20x1.40mm_HandSolder -> Resistor_SMD:R_0805_2012Metric; MFG Part No. (none) -> RMCF0805FT64K9
- R65: renamed from R53; footprint Resistor_SMD:R_0805_2012Metric_Pad1.20x1.40mm_HandSolder -> Resistor_SMD:R_0805_2012Metric; MFG Part No. (none) -> RMCF0805FT100K
- R66: renamed from R54; footprint Resistor_SMD:R_1206_3216Metric_Pad1.30x1.75mm_HandSolder -> Resistor_SMD:R_0805_2012Metric; MFG Part No. (none) -> RMCF0805FT240K
- R67: renamed from R55; footprint Resistor_SMD:R_0805_2012Metric_Pad1.20x1.40mm_HandSolder -> Resistor_SMD:R_0805_2012Metric; MFG Part No. (none) -> RMCF0805FT56K0
- R68: renamed from R56; footprint Resistor_SMD:R_0805_2012Metric_Pad1.20x1.40mm_HandSolder -> Resistor_SMD:R_0805_2012Metric; MFG Part No. (none) -> RMCF0805FT4K70
- R69: renamed from R57; footprint Resistor_SMD:R_0805_2012Metric_Pad1.20x1.40mm_HandSolder -> Resistor_SMD:R_0805_2012Metric; MFG Part No. (none) -> RMCF0805FT4K70
- U10: renamed from U8; MFG Part No. (none) -> MCP4728-E/UN
- U9: renamed from U7; MFG Part No. (none) -> MCP6002-I/SN
Connections:
- net +3.3VA: no longer C31.2, U10.1 (VDD)
- net SERCOM4[0] renamed dac-sda
- net SERCOM4[1] renamed dac-scl
- new net +5V: C31.2, U10.1 (VDD)
