File: profane_geometry/mcu.sch (KiCad schematic (older format))
At the start: 5 parts

Commit message: update .gitignore, current kicad project
Parts:
- removed C?: 1uF, symbol Device:C
- removed C? (x2): 0.1uF, symbol Device:C
- removed SW?: SW_SPST, symbol Switch:SW_SPST
- removed U?: ATSAMD21E18A-A, Package_QFP:TQFP-32_7x7mm_P0.8mm, symbol MCU_Microchip_SAMD:ATSAMD21E18A-A
- added C32: 1uF, Capacitor_SMD:C_0805_2012Metric, symbol Device:C
- added C33, C34, C35, C36, C37: 0.1uF, Capacitor_SMD:C_0805_2012Metric, symbol Device:C
- added D1: PWR, zzzzzzzz:SunLED-Rev-2-PLCC-SeeThru, symbol Device:LED
- added J3: USB_B_Micro, Connector_USB:USB_Micro-B_Amphenol_10103594-0001LF_Horizontal, symbol Connector:USB_B_Micro
- added J4: TagConect SWD, Connector:Tag-Connect_TC2030-IDC-NL_2x03_P1.27mm_Vertical, symbol Connector_Generic:Conn_02x03_Counter_Clockwise
- added NT1: GND_Net_Tie, NetTie:NetTie-2_SMD_Pad0.5mm, symbol Device:Net-Tie_2
- added R1: 330R, Resistor_SMD:R_0805_2012Metric, symbol Device:R_US
- added R70, R71: 4.7k, Resistor_SMD:R_0805_2012Metric, symbol Device:R_US
- added SW1: RESET_SW, zzzzzzzz:SPST_TL3365AF180QG_SMD, symbol Switch:SW_MEC_5E
- added TP10: PSL, TestPoint:TestPoint_Pad_D1.0mm, symbol Connector:TestPoint
- added TP11: NSL, TestPoint:TestPoint_Pad_D1.0mm, symbol Connector:TestPoint
- added TP12: D_SDA, TestPoint:TestPoint_Pad_D1.0mm, symbol Connector:TestPoint
- added TP13: D_SCL, TestPoint:TestPoint_Pad_D1.0mm, symbol Connector:TestPoint
- added TP14: L_SDA, TestPoint:TestPoint_Pad_D1.0mm, symbol Connector:TestPoint
- added TP15: L_SCL, TestPoint:TestPoint_Pad_D1.0mm, symbol Connector:TestPoint
- added TP5: V/OCT, TestPoint:TestPoint_Pad_D1.0mm, symbol Connector:TestPoint
- added TP6: PWM, TestPoint:TestPoint_Pad_D1.0mm, symbol Connector:TestPoint
- added TP7: POT, TestPoint:TestPoint_Pad_D1.0mm, symbol Connector:TestPoint
- added TP8: TSL, TestPoint:TestPoint_Pad_D1.0mm, symbol Connector:TestPoint
- added TP9: SSL, TestPoint:TestPoint_Pad_D1.0mm, symbol Connector:TestPoint
- added U11: ATSAMD21G18A-AUT, Package_QFP:TQFP-48_7x7mm_P0.5mm, symbol MCU_Microchip_SAMD:ATSAMD21G18A-AUT
Connections:
- net +3.3VA: now also C36.2, U11.6 (VDDANA)
- net +3V3: now also C34.2, C35.2, C37.2, J4.1 (Pin_1), R70.2, R71.2, U11.17 (VDDIO), U11.36 (VDDIO), U11.44 (VDDIN)
- net GND: now also C32.1, C33.1, C34.1, C35.1, C36.1, C37.1, D1.1 (K), J3.4 (ID), J4.5 (Pin_5), NT1.2, SW1.3 (K), SW1.4 (A), U11.18 (GND), U11.35 (GND), U11.42 (GND), U11.5 (GNDANA)
- net RESET: now also J4.3 (Pin_3), SW1.1, SW1.2, U11.40 (~RESET)
- new net: C32.2, U11.43 (VDDCORE)
- new net: D1.2 (A), R1.2
- new net AIN[1](VREFA): C33.2, U11.4 (PA03)
- new net AIN[6]: U11.11 (PA06)
- new net AIN[7]: U11.12 (PA07)
- new net D+: J3.3 (D+), U11.34 (PA25)
- new net D-: J3.2 (D-), U11.33 (PA24)
- new net GNDD: J3.5 (GND), NT1.1
- new net SWCLK: J4.4 (Pin_4), U11.45 (PA30)
- new net SWDIO: J4.2 (Pin_2), U11.46 (PA31)
- new net TCC0_WO[6]: R1.1, U11.29 (PA20)
- new net dac-scl: TP13.1, U11.22 (PA13)
- new net dac-sda: TP12.1, U11.21 (PA12)
- new net notch-slider-led: TP11.1, U11.20 (PB11)
- new net pulse-slider-led: TP10.1, U11.19 (PB10)
- new net pwm-pot: TP7.1, U11.10 (PA05)
- new net pwm-scaled: TP6.1, U11.9 (PA04)
- new net rgb-scl: R71.1, TP15.1, U11.26 (PA17)
- new net rgb-sda: R70.1, TP14.1, U11.25 (PA16)
- new net square-slider-led: TP9.1, U11.16 (PA11)
- new net tri-slider-led: TP8.1, U11.15 (PA10)
- new net v-oct-scaled: TP5.1, U11.3 (PA02)
- no-connect marks 0 -> 24
Other:
- note added: "Analog Ins/VREF"
- note added: "DEBUG"
- note added: "I2C - DAC"
- note added: "I2C - RGB"
- note added: "Power LED"
- note added: "Satisfies the ERC - The USB micro symbol here considers\nGND to be a Power Output pin, meaning we can't just tie our \nown GND to it directly. Instead KiCad can accomplish joining\nof ground planes via this special Net Tie symbol. In practice\nthis appears to just give us a copper trace we can use to "join"\nthe two ground planes on the PCB"
- note added: "Slider LED PWM"
- note added: "USB"
