File: profane_geometry/mixer.sch (KiCad schematic (older format))
At the start: 23 parts, among them U5 TL074, U6 TL072

Commit message: update .gitignore, current kicad project
Parts:
- removed C15: 8.2pF, Capacitor_SMD:C_0805_2012Metric_Pad1.18x1.45mm_HandSolder, symbol Device:C
- removed R34: 20k, Resistor_SMD:R_0805_2012Metric_Pad1.20x1.40mm_HandSolder, symbol Device:R_US
- removed unit 1 of U6
- added C18, C19, C20, C21: 47pF, Capacitor_SMD:C_0805_2012Metric, symbol Device:C
- added C26, C27: 0.1uF, Capacitor_SMD:C_0805_2012Metric, symbol Device:C
- added R40, R45, R51, R52, R57: 10k, Resistor_SMD:R_0805_2012Metric, symbol Device:R_US
- added R43, R55: 2.2M, Resistor_SMD:R_0805_2012Metric, symbol Device:R_US
- added R50, R56: 30.1k, Resistor_SMD:R_0805_2012Metric, symbol Device:R_US
- added R53, R58: 22k, Resistor_SMD:R_0805_2012Metric, symbol Device:R_US
- added R54: 47k, Resistor_SMD:R_0805_2012Metric, symbol Device:R_US
- added U7: TL074, Package_SO:SSOP-14_5.3x6.2mm_P0.65mm, symbol Amplifier_Operational:TL074
- C22: renamed from C16; footprint Capacitor_SMD:C_1206_3216Metric_Pad1.33x1.80mm_HandSolder -> Capacitor_SMD:C_0805_2012Metric; MFG Part No. (none) -> 08055C104KAT4A
- C23: renamed from C17; footprint Capacitor_SMD:C_1206_3216Metric_Pad1.33x1.80mm_HandSolder -> Capacitor_SMD:C_0805_2012Metric; MFG Part No. (none) -> 08055C104KAT4A
- C24: renamed from C22; footprint Capacitor_SMD:C_1206_3216Metric_Pad1.33x1.80mm_HandSolder -> Capacitor_SMD:C_0805_2012Metric; MFG Part No. (none) -> 08055C104KAT4A
- C25: renamed from C23; footprint Capacitor_SMD:C_1206_3216Metric_Pad1.33x1.80mm_HandSolder -> Capacitor_SMD:C_0805_2012Metric; MFG Part No. (none) -> 08055C104KAT4A
- R35: value 20k -> 10k; footprint Resistor_SMD:R_0805_2012Metric_Pad1.20x1.40mm_HandSolder -> Resistor_SMD:R_0805_2012Metric; MFG Part No. (none) -> RMCF0805FT10K0
- R36, R48: value 20k -> 2.2M; footprint Resistor_SMD:R_0805_2012Metric_Pad1.20x1.40mm_HandSolder -> Resistor_SMD:R_0805_2012Metric; MFG Part No. (none) -> RMCF0805FT2M20
- R37: value 100k -> 47k; footprint Resistor_SMD:R_0805_2012Metric_Pad1.20x1.40mm_HandSolder -> Resistor_SMD:R_0805_2012Metric; MFG Part No. (none) -> RMCF0805FT47K0
- R38: value 20k -> 30.1k; footprint Resistor_SMD:R_0805_2012Metric_Pad1.20x1.40mm_HandSolder -> Resistor_SMD:R_0805_2012Metric; MFG Part No. (none) -> RMCF0805FT30K1
- R39, R47: value 100k -> 10k; footprint Resistor_SMD:R_0805_2012Metric_Pad1.20x1.40mm_HandSolder -> Resistor_SMD:R_0805_2012Metric; MFG Part No. (none) -> RMCF0805FT10K0
- R41: value 100k -> 22k; footprint Resistor_SMD:R_0805_2012Metric_Pad1.20x1.40mm_HandSolder -> Resistor_SMD:R_0805_2012Metric; MFG Part No. (none) -> RMCF0805FT22K0
- R42, R49: value 20k -> 47k; footprint Resistor_SMD:R_0805_2012Metric_Pad1.20x1.40mm_HandSolder -> Resistor_SMD:R_0805_2012Metric; MFG Part No. (none) -> RMCF0805FT47K0
- R44: value 100k -> 30.1k; footprint Resistor_SMD:R_0805_2012Metric_Pad1.20x1.40mm_HandSolder -> Resistor_SMD:R_0805_2012Metric; MFG Part No. (none) -> RMCF0805FT30K1
- R46: value 20k -> 22k; footprint Resistor_SMD:R_0805_2012Metric_Pad1.20x1.40mm_HandSolder -> Resistor_SMD:R_0805_2012Metric; MFG Part No. (none) -> RMCF0805FT22K0
- R59: renamed from R40; value 20k -> 10k; footprint Resistor_SMD:R_0805_2012Metric_Pad1.20x1.40mm_HandSolder -> Resistor_SMD:R_0805_2012Metric; MFG Part No. (none) -> RMCF0805FT10K0
- R60: renamed from R43; value 20k -> 10k; footprint Resistor_SMD:R_0805_2012Metric_Pad1.20x1.40mm_HandSolder -> Resistor_SMD:R_0805_2012Metric; MFG Part No. (none) -> RMCF0805FT10K0
- R61: renamed from R45; footprint Resistor_SMD:R_0805_2012Metric_Pad1.20x1.40mm_HandSolder -> Resistor_SMD:R_0805_2012Metric; MFG Part No. (none) -> RMCF0805FT1K00
- U6: renamed from U5; footprint Package_SO:SOIC-14_3.9x8.7mm_P1.27mm -> Package_SO:SSOP-14_5.3x6.2mm_P0.65mm; MFG Part No. (none) -> TL074CDBR
- U8: renamed from U6; MFG Part No. (none) -> TL072QDREP
Connections:
- net mix-att is gone; now on net GND: U8.5 (+)
- net notch-att-in is gone; now on net GND: U6.12 (+)
- net tri-att-in is gone; now on net GND: U6.3 (+)
- net +12V: now also C26.1, U7.4 (V+)
- net -12V: now also C27.2, U7.11 (V-)
- net GND: now also R41.1, R46.1, C26.2, C27.1, R53.1, R58.1, U7.12 (+), U7.3 (+)
- net notch-in: now also R44.2; no longer R49.2
- net pulse-in: now also R56.2; no longer R46.2
- net square-in: now also R50.2; no longer R38.2
- net tri-in: now also R38.2; no longer R35.2
- net at R37.2: now also R36.1, R41.2, U6.6 (-), C18.2; no longer U6.1
- net at U6.2 (-): now also R35.2, R38.1; no longer R35.1
- net mix-pre renamed notch-ch
- net notch-ch: now also R45.2, R51.1, R57.2
- net pulse-att-in renamed sq-mix-in
- net square-att-in renamed tri-mix-in
- new net: C18.1, R37.1, R39.2, U6.7
- new net: C20.1, R49.1, R51.2, U6.8
- new net: C20.2, R48.1, R49.2, R53.2, U6.9 (-)
- new net: R47.2, R50.1, U6.13 (-)
- new net: R40.2, R44.1, U7.2 (-)
- new net: C19.2, R42.2, R43.1, R46.2, U7.6 (-)
- new net: C19.1, R42.1, R45.1, U7.7
- new net: C21.1, R54.1, R57.1, U7.8
- new net: C21.2, R54.2, R55.1, R58.2, U7.9 (-)
- new net: R52.2, R56.1, U7.13 (-)
- new net nt-mix-in: U7.5 (+)
- new net nt-pre-mix: R40.1, R43.2, U7.1
- new net pl-mix-in: U7.10 (+)
- new net pl-pre-mix: R52.1, R55.2, U7.14
- new net sq-pre-mix: R47.1, R48.2, U6.14
- new net tri-pre-mix: R35.1, R36.2, U6.1
Other:
- note added: "Individual channel level\nEach channel out goes through an inverting amp with a gain of -0.333\nbefore being sent out to the slide pots on the jackboard, the large resistor\nand following non-inverting amp (with a gain of approx +3) are to \nimpove the offness of the slide pots, since they're low-cost non-inifinity-off components"
- note added: "Top / wiper of slide pot"
- moved on the sheet: R59, R60, R61, U6A, U6B, U6C, U6D, U8B
