File: profane_geometry/power.sch (KiCad schematic (older format))
At the start: 9 parts, among them U1 LM1117-3.3

Commit message: update .gitignore, current kicad project
Parts:
- added C4, C6: 1uF, Capacitor_SMD:C_0805_2012Metric, symbol Device:C
- added U2: AP2112K-3.3, Package_TO_SOT_SMD:SOT-23-5, symbol Regulator_Linear:AP2112K-3.3
- C1, C2: MFG Part No. (none) -> 35SVPK47M
- C3: footprint Capacitor_SMD:C_1206_3216Metric_Pad1.33x1.80mm_HandSolder -> Capacitor_SMD:C_0805_2012Metric; MFG Part No. (none) -> 08055C104KAT4A
- D2: renamed from D1; MFG Part No. (none) -> 1N5819HWQ-7-F
- D3: renamed from D2; MFG Part No. (none) -> 1N5819HWQ-7-F
- FB1, FB2, FB3: MFG Part No. (none) -> 742792312
- U1: value LM1117-3.3 -> LM1117-5; MFG Part No. (none) -> LM1117MP-5.0/NOPB
Connections:
- net +3V3: now also C6.1, U2.5 (VOUT); no longer C2.1, C3.1, U1.2 (VO)
- net GND: now also C4.2, C6.2, U2.2 (GND)
- new net +5V: C2.1, C3.1, C4.1, U1.2 (VO), U2.1 (VIN), U2.3 (EN)
Other:
- note added: "If I put a diode here and then attach the USB port's\nVBUS line to the +5V power rail, considering the 5V\nnet attaches only to the 3.3v regulator and the\nDAC, can I effectively power the board via usb for\ndebugging/flashing without needing rack power?"
- moved on the sheet: D2, FB1, FB2
