File: profane_geometry/profane_geometry.sch (KiCad schematic (older format))
At the start: 2 parts, among them J1 Conn_01x12, J2 Conn_01x12

Commit message: update .gitignore, current kicad project
Parts:
- removed J1, J2: Conn_01x12, Connector_PinSocket_2.54mm:PinSocket_1x12_P2.54mm_Vertical, symbol Connector_Generic:Conn_01x12
- added J1, J2: Conn_02x08_Odd_Even, Connector_PinHeader_2.54mm:PinHeader_2x08_P2.54mm_Vertical, symbol Connector_Generic:Conn_02x08_Odd_Even
Connections:
- net +12v-rack: now also J2.3 (Pin_3)
- net +3V3: now also J2.12 (Pin_12)
- net -12v-rack: now also J2.1 (Pin_1)
- net GND: now also J1.15 (Pin_15), J1.16 (Pin_16), J2.15 (Pin_15), J2.16 (Pin_16)
- net mix-out: now also J2.13 (Pin_13)
- net notch-out: now also J1.1 (Pin_1)
- net pulse-cv: now also J2.7 (Pin_7)
- net pulse-out: now also J1.3 (Pin_3)
- net square-out: now also J1.2 (Pin_2)
- net tri-out: now also J1.4 (Pin_4)
- net v_oct-cv: now also J2.5 (Pin_5)
- new net notch-mix-in: J1.9 (Pin_9)
- new net notch-pre-out: J1.5 (Pin_5)
- new net notch-slider-led: J2.8 (Pin_8)
- new net pulse-mix-in: J1.11 (Pin_11)
- new net pulse-pot-in: J2.11 (Pin_11)
- new net pulse-pre-out: J1.7 (Pin_7)
- new net pulse-slider-led: J2.6 (Pin_6)
- new net rgb-scl: J2.10 (Pin_10)
- new net rgb-sda: J2.9 (Pin_9)
- new net square-mix-in: J1.10 (Pin_10)
- new net square-pre-out: J1.6 (Pin_6)
- new net square-slider-led: J2.4 (Pin_4)
- new net tri-mix-in: J1.12 (Pin_12)
- new net tri-pre-out: J1.8 (Pin_8)
- new net tri-slider-led: J2.2 (Pin_2)
- no-connect marks 2 -> 3
Other:
- note added: "Profane Geometry (aka. Demon Core)"
- note added: "v0.3 9/12/21"
- note removed: "Profane Geometry"
