File: profane_geometry_jackboard/profane_geometry_jackboard.sch (KiCad schematic (older format))
At the start: 21 parts, among them J1 TriAmt, J11 NotchOut, J12 PulseAmt, J13 V/OCT, J14 PulseCV, J15 MixOut, J2 TriOut, J3 Conn_02x08_Counter_Clockwise, J4 Conn_01x12, J5 SquareAmt, J6 SquareOut, J7 Conn_01x12, J8 PulseOut, J9 PulseAmt

Commit message: update .gitignore, current kicad project
Parts:
- removed A1: Adafruit_Feather_M0_Express, profane_geometry_jackboard:Adafruit_Feather_M0_Express, symbol zzzzzzzz:Adafruit_Feather_M0_Express
- removed J1: TriAmt, profane_geometry_jackboard:Jack_3.5mm_QingPu_WQP-PJ301BM_Vertical, symbol Connector:AudioJack2_SwitchT
- removed J12, J9: PulseAmt, profane_geometry_jackboard:Jack_3.5mm_QingPu_WQP-PJ301BM_Vertical, symbol Connector:AudioJack2_SwitchT
- removed J3: Conn_02x08_Counter_Clockwise, profane_geometry_jackboard:Molex_02x08_2.54mm_Shrouded_Keyed, symbol Connector_Generic:Conn_02x08_Counter_Clockwise
- removed J4, J7: Conn_01x12, Connector_PinHeader_2.54mm:PinHeader_1x12_P2.54mm_Vertical, symbol Connector_Generic:Conn_01x12
- removed J5: SquareAmt, profane_geometry_jackboard:Jack_3.5mm_QingPu_WQP-PJ301BM_Vertical, symbol Connector:AudioJack2_SwitchT
- removed RV1: MixAtt, Potentiometer_THT:Potentiometer_TT_P0915N, symbol Device:R_POT_US
- added D1, D2, D3, D4, D5, D6, D7, D8: APA102-2020, LED_SMD:LED-APA102-2020, symbol LED:APA102-2020
- added J1, J3: Conn_02x08_Odd_Even, Connector_PinSocket_2.54mm:PinSocket_2x08_P2.54mm_Vertical, symbol Connector_Generic:Conn_02x08_Odd_Even
- added J4: Conn_02x05_Odd_Even, Connector_PinHeader_2.54mm:PinHeader_2x05_P2.54mm_Vertical, symbol Connector_Generic:Conn_02x05_Odd_Even
Connections:
- net +12v-rack: now also J3.3 (Pin_3), J4.1 (Pin_1), J4.2 (Pin_2)
- net +3V3: now also RV2.3, D1.1 (VDD), D2.1 (VDD), D3.1 (VDD), D4.1 (VDD), D5.1 (VDD), D6.1 (VDD), D7.1 (VDD), D8.1 (VDD), J3.12 (Pin_12); no longer RV2.1
- net -12v-rack: now also J3.1 (Pin_1), J4.10 (Pin_10), J4.9 (Pin_9)
- net GND: now also RV2.1, D1.6 (GND), D2.6 (GND), D3.6 (GND), D4.6 (GND), D5.6 (GND), D6.6 (GND), D7.6 (GND), D8.6 (GND), J1.15 (Pin_15), J1.16 (Pin_16), J3.15 (Pin_15), J3.16 (Pin_16), J4.3 (Pin_3), J4.4 (Pin_4), J4.5 (Pin_5), J4.6 (Pin_6), J4.7 (Pin_7), J4.8 (Pin_8); no longer RV2.3
- net mix-out: now also J3.13 (Pin_13)
- net notch-out: now also J1.1 (Pin_1)
- net pulse-cv: now also J3.7 (Pin_7)
- net pulse-out: now also J1.3 (Pin_3)
- net pulse-pot: now also J3.11 (Pin_11)
- net square-out: now also J1.2 (Pin_2)
- net tri-out: now also J1.4 (Pin_4)
- net v_oct-cv: now also J3.5 (Pin_5)
- net notch-pre-out: now reaches VR4.3 (CW)
- net notch-pre-out: now also J1.5 (Pin_5)
- net pulse-pre-out: now reaches VR3.3 (CW)
- net pulse-pre-out: now also J1.7 (Pin_7)
- net square-pre-out: now reaches VR2.3 (CW)
- net square-pre-out: now also J1.6 (Pin_6)
- net tri-pre-out: now reaches VR1.3 (CW)
- net tri-pre-out: now also J1.8 (Pin_8)
- net notch-att renamed notch-mix
- net notch-mix: now also J1.9 (Pin_9)
- net notch-led renamed notch-slider-led
- net notch-slider-led: now also J3.8 (Pin_8)
- net pulse-att renamed pulse-mix
- net pulse-mix: now also J1.11 (Pin_11)
- net pulse-led renamed pulse-slider-led
- net pulse-slider-led: now also J3.6 (Pin_6)
- net square-att renamed square-mix
- net square-mix: now also J1.10 (Pin_10)
- net square-led renamed square-slider-led
- net square-slider-led: now also J3.4 (Pin_4)
- net tri-att renamed tri-mix
- net tri-mix: now also J1.12 (Pin_12)
- net tri-led renamed tri-slider-led
- net tri-slider-led: now also J3.2 (Pin_2)
- new net: D1.2 (CKO), D2.5 (CKI)
- new net: D1.3 (SDO), D2.4 (SDI)
- new net: D2.2 (CKO), D3.5 (CKI)
- new net: D2.3 (SDO), D3.4 (SDI)
- new net: D3.2 (CKO), D4.5 (CKI)
- new net: D3.3 (SDO), D4.4 (SDI)
- new net: D4.2 (CKO), D5.5 (CKI)
- new net: D4.3 (SDO), D5.4 (SDI)
- new net: D5.2 (CKO), D6.5 (CKI)
- new net: D5.3 (SDO), D6.4 (SDI)
- new net: D6.2 (CKO), D7.5 (CKI)
- new net: D6.3 (SDO), D7.4 (SDI)
- new net: D7.2 (CKO), D8.5 (CKI)
- new net: D7.3 (SDO), D8.4 (SDI)
- new net rgb-scl: D1.5 (CKI), J3.10 (Pin_10)
- new net rgb-sda: D1.4 (SDI), J3.9 (Pin_9)
- no-connect marks 16 -> 12
Other:
- note added: "v0.3 9/12/21"
- moved on the sheet: J11, J13, J14, J15, J2, J6, J8, RV2, VR1, VR2, VR3, VR4
